Commit message: HH_Ver2

File: Olaf_bot/Olaf_description/urdf/Olaf.urdf.xacro (robot description, xacro)
@@ -1,5 +1,5 @@
 <?xml version="1.0" ?>
-<robot name="omo_r1" xmlns:xacro="http://ros.org/wiki/xacro">
-  <xacro:include filename="$(find omo_r1_description)/urdf/common_properties.xacro"/>
+<robot name="Olaf" xmlns:xacro="http://ros.org/wiki/xacro">
+  <xacro:include filename="$(find Olaf_description)/urdf/common_properties.xacro"/>
   <link name="base_footprint"/>
   <joint name="base_joint" type="fixed">
@@ -12,5 +12,5 @@
       <origin xyz="0.097 0.276 0.19" rpy="3.14 0 -1.57"/>
       <geometry>
-        <mesh filename="package://omo_r1_description/meshes/bases/omo_r1_body.stl" scale="0.001 0.001 0.001"/>
+        <mesh filename="package://Olaf_description/meshes/bases/Olaf_body.stl" scale="0.001 0.001 0.001"/>
       </geometry>
       <material name="light_black"/>
@@ -19,5 +19,5 @@
       <origin xyz="0.097 0.276 0.19" rpy="3.14 0 -1.57"/>
       <geometry>
-        <mesh filename="package://omo_r1_description/meshes/bases/omo_r1_body.stl" scale="0.001 0.001 0.001"/>
+        <mesh filename="package://Olaf_description/meshes/bases/Olaf_body.stl" scale="0.001 0.001 0.001"/>
       </geometry>
     </collision>
@@ -40,5 +40,5 @@
       <origin xyz="-0.1105 -0.06 0.1104" rpy="-1.57 0 0"/>
       <geometry>
-        <mesh filename="package://omo_r1_description/meshes/wheels/omo_r1_wheel.stl" scale="0.001 0.001 0.001"/>
+        <mesh filename="package://Olaf_description/meshes/wheels/Olaf_wheel.stl" scale="0.001 0.001 0.001"/>
       </geometry>
       <material name="dark"/>
@@ -47,5 +47,5 @@
       <origin xyz="-0.1105 -0.06 0.1104" rpy="-1.57 0 0"/>
       <geometry>
-        <mesh filename="package://omo_r1_description/meshes/wheels/omo_r1_wheel.stl" scale="0.001 0.001 0.001"/>
+        <mesh filename="package://Olaf_description/meshes/wheels/Olaf_wheel.stl" scale="0.001 0.001 0.001"/>
       </geometry>
     </collision>
@@ -68,5 +68,5 @@
       <origin xyz="-0.110 0.06 -0.1103" rpy="1.57 0 0"/>
       <geometry>
-        <mesh filename="package://omo_r1_description/meshes/wheels/omo_r1_wheel.stl" scale="0.001 0.001 0.001"/>
+        <mesh filename="package://Olaf_description/meshes/wheels/Olaf_wheel.stl" scale="0.001 0.001 0.001"/>
       </geometry>
       <material name="dark"/>
@@ -75,5 +75,5 @@
       <origin xyz="-0.110 0.06 -0.1103" rpy="1.57 0 0"/>
       <geometry>
-        <mesh filename="package://omo_r1_description/meshes/wheels/omo_r1_wheel.stl" scale="0.001 0.001 0.001"/>
+        <mesh filename="package://Olaf_description/meshes/wheels/Olaf_wheel.stl" scale="0.001 0.001 0.001"/>
       </geometry>
     </collision>
@@ -141,5 +141,5 @@
       <origin xyz="0 0 0.0" rpy="0.0 0 0.0"/>
       <geometry>
-        <mesh filename="package://omo_r1_description/meshes/sensors/omo_r1_lidar.stl" scale="0.001 0.001 0.001"/>
+        <mesh filename="package://Olaf_description/meshes/sensors/Olaf_lidar.stl" scale="0.001 0.001 0.001"/>
       </geometry>
       <material name="dark"/>
@@ -148,5 +148,5 @@
       <origin xyz="0 0 0.0" rpy="0.0 0 0.0"/>
       <geometry>
-        <mesh filename="package://omo_r1_description/meshes/sensors/omo_r1_lidar.stl" scale="0.001 0.001 0.001"/>
+        <mesh filename="package://Olaf_description/meshes/sensors/Olaf_lidar.stl" scale="0.001 0.001 0.001"/>
       </geometry>
     </collision>
@@ -168,5 +168,5 @@
       <origin xyz="0 0 0.0" rpy="1.5758 0.0 1.5758"/>
       <geometry>
-        <mesh filename="package://omo_r1_description/meshes/sensors/omo_r1_camera.stl" scale="0.001 0.001 0.001"/>
+        <mesh filename="package://Olaf_description/meshes/sensors/Olaf_camera.stl" scale="0.001 0.001 0.001"/>
       </geometry>
       <material name="dark"/>
@@ -175,5 +175,5 @@
       <origin xyz="0 0 0.0" rpy="1.5758 0.0 1.5758"/>
       <geometry>
-        <mesh filename="package://omo_r1_description/meshes/sensors/omo_r1_camera.stl" scale="0.001 0.001 0.001"/>
+        <mesh filename="package://Olaf_description/meshes/sensors/Olaf_camera.stl" scale="0.001 0.001 0.001"/>
       </geometry>
     </collision>

File: Olaf_bot/Olaf_gazebo/sdf/Olaf.gazebo.xacro (robot description, xacro)
@@ -1,5 +1,5 @@
 <?xml version="1.0"?>
-<robot name="omo_r1_sim" xmlns:xacro="http://ros.org/wiki/xacro">
-  <xacro:include filename="$(find omo_r1_description)/urdf/omo_r1.urdf.xacro"/>
+<robot name="Olaf_sim" xmlns:xacro="http://ros.org/wiki/xacro">
+  <xacro:include filename="$(find Olaf_description)/urdf/Olaf.urdf.xacro"/>
   <xacro:arg name="laser_visual"  default="false"/>
   <xacro:arg name="camera_visual" default="false"/>
@@ -54,5 +54,5 @@
   </gazebo>
   <gazebo>
-    <plugin name="omo_r1_controller" filename="libgazebo_ros_diff_drive.so">
+    <plugin name="Olaf_controller" filename="libgazebo_ros_diff_drive.so">
       <commandTopic>cmd_vel</commandTopic>
       <odometryTopic>odom</odometryTopic>
