Commit message: HH_ver.01

File: Olaf_bot/Olaf_description/urdf/Olaf.urdf.g2.xacro (robot description, xacro)
@@ -1,5 +1,5 @@
 <?xml version="1.0" ?>
-<robot name="omo_r1" xmlns:xacro="http://ros.org/wiki/xacro">
-  <xacro:include filename="$(find omo_r1_description)/urdf/common_properties.xacro"/>
+<robot name="Olaf" xmlns:xacro="http://ros.org/wiki/xacro">
+  <xacro:include filename="$(find Olaf_description)/urdf/common_properties.xacro"/>
   <link name="base_footprint"/>
   <joint name="base_joint" type="fixed">
@@ -12,5 +12,5 @@
       <origin xyz="0.097 0.276 0.19" rpy="3.14 0 -1.57"/>
       <geometry>
-        <mesh filename="package://omo_r1_description/meshes/bases/omo_r1_body.stl" scale="0.001 0.001 0.001"/>
+        <mesh filename="package://Olaf_description/meshes/bases/Olaf_body.stl" scale="0.001 0.001 0.001"/>
       </geometry>
       <material name="light_black"/>
@@ -19,5 +19,5 @@
       <origin xyz="0.097 0.276 0.19" rpy="3.14 0 -1.57"/>
       <geometry>
-        <mesh filename="package://omo_r1_description/meshes/bases/omo_r1_body.stl" scale="0.001 0.001 0.001"/>
+        <mesh filename="package://Olaf_description/meshes/bases/Olaf_body.stl" scale="0.001 0.001 0.001"/>
       </geometry>
     </collision>
@@ -40,5 +40,5 @@
       <origin xyz="-0.1105 -0.06 0.1104" rpy="-1.57 0 0"/>
       <geometry>
-        <mesh filename="package://omo_r1_description/meshes/wheels/omo_r1_wheel.stl" scale="0.001 0.001 0.001"/>
+        <mesh filename="package://Olaf_description/meshes/wheels/Olaf_wheel.stl" scale="0.001 0.001 0.001"/>
       </geometry>
       <material name="dark"/>
@@ -47,5 +47,5 @@
       <origin xyz="-0.1105 -0.06 0.1104" rpy="-1.57 0 0"/>
       <geometry>
-        <mesh filename="package://omo_r1_description/meshes/wheels/omo_r1_wheel.stl" scale="0.001 0.001 0.001"/>
+        <mesh filename="package://Olaf_description/meshes/wheels/Olaf_wheel.stl" scale="0.001 0.001 0.001"/>
       </geometry>
     </collision>
@@ -68,5 +68,5 @@
       <origin xyz="-0.110 0.06 -0.1103" rpy="1.57 0 0"/>
       <geometry>
-        <mesh filename="package://omo_r1_description/meshes/wheels/omo_r1_wheel.stl" scale="0.001 0.001 0.001"/>
+        <mesh filename="package://Olaf_description/meshes/wheels/Olaf_wheel.stl" scale="0.001 0.001 0.001"/>
       </geometry>
       <material name="dark"/>
@@ -75,5 +75,5 @@
       <origin xyz="-0.110 0.06 -0.1103" rpy="1.57 0 0"/>
       <geometry>
-        <mesh filename="package://omo_r1_description/meshes/wheels/omo_r1_wheel.stl" scale="0.001 0.001 0.001"/>
+        <mesh filename="package://Olaf_description/meshes/wheels/Olaf_wheel.stl" scale="0.001 0.001 0.001"/>
       </geometry>
     </collision>
@@ -141,5 +141,5 @@
       <origin xyz="0 0 0.0" rpy="0.0 0 0.0"/>
       <geometry>
-        <mesh filename="package://omo_r1_description/meshes/sensors/omo_r1_lidar.stl" scale="0.001 0.001 0.001"/>
+        <mesh filename="package://Olaf_description/meshes/sensors/Olaf_lidar.stl" scale="0.001 0.001 0.001"/>
       </geometry>
       <material name="dark"/>
@@ -148,5 +148,5 @@
       <origin xyz="0 0 0.0" rpy="0.0 0 0.0"/>
       <geometry>
-        <mesh filename="package://omo_r1_description/meshes/sensors/omo_r1_lidar.stl" scale="0.001 0.001 0.001"/>
+        <mesh filename="package://Olaf_description/meshes/sensors/Olaf_lidar.stl" scale="0.001 0.001 0.001"/>
       </geometry>
     </collision>
@@ -168,5 +168,5 @@
       <origin xyz="0 0 0.0" rpy="1.5758 0.0 1.5758"/>
       <geometry>
-        <mesh filename="package://omo_r1_description/meshes/sensors/omo_r1_camera.stl" scale="0.001 0.001 0.001"/>
+        <mesh filename="package://Olaf_description/meshes/sensors/Olaf_camera.stl" scale="0.001 0.001 0.001"/>
       </geometry>
       <material name="dark"/>
@@ -175,5 +175,5 @@
       <origin xyz="0 0 0.0" rpy="1.5758 0.0 1.5758"/>
       <geometry>
-        <mesh filename="package://omo_r1_description/meshes/sensors/omo_r1_camera.stl" scale="0.001 0.001 0.001"/>
+        <mesh filename="package://Olaf_description/meshes/sensors/Olaf_camera.stl" scale="0.001 0.001 0.001"/>
       </geometry>
     </collision>

Commit message: 11.12 fail ekf

File: Olaf_bot/Olaf_description/urdf/Olaf.urdf.g2.xacro (robot description, xacro)
@@ -126,10 +126,10 @@
     </inertial>
   </link>
-  <joint name="imu_joint" type="fixed">
+  <!-- <joint name="imu_joint" type="fixed">
     <parent link="base_link"/>
     <child link="imu_link"/>
     <origin xyz="0.0 0 0.190" rpy="0 0 1.5758"/>
   </joint>
-  <link name="imu_link"/>
+  <link name="imu_link"/> -->
   <joint name="scan_joint" type="fixed">
     <parent link="base_link"/>

Commit message: 11.15 plus map

File: Olaf_bot/Olaf_description/urdf/Olaf.urdf.g2.xacro (robot description, xacro)
@@ -2,10 +2,10 @@
 <robot name="Olaf" xmlns:xacro="http://ros.org/wiki/xacro">
   <xacro:include filename="$(find Olaf_description)/urdf/common_properties.xacro"/>
-  <link name="base_footprint"/>
+  <!-- <link name="base_footprint"/>
   <joint name="base_joint" type="fixed">
     <parent link="base_footprint"/>
     <child link="base_link" />
     <origin xyz="0 0.0 0.07" rpy="0 0 0.0"/>
-  </joint>
+  </joint> -->
   <link name="base_link">
     <visual>

File: Olaf_bot/Olaf_description/urdf/Olaf.urdf.xacro (robot description, xacro)
@@ -1,3 +1,3 @@
-<?xml version="1.0" ?>
+<!-- <?xml version="1.0" ?>
 <robot name="Olaf" xmlns:xacro="http://ros.org/wiki/xacro">
   <xacro:include filename="$(find Olaf_description)/urdf/common_properties.xacro"/>
@@ -191,3 +191,3 @@
   </joint>
   <link name="camera_rgb_optical_frame"/>
-</robot>
+</robot> -->

Commit message: add map and map TF

File: Olaf_bot/Olaf_description/urdf/Olaf.urdf.g2.xacro (robot description, xacro)
@@ -5,8 +5,8 @@
   <joint name="base_joint" type="fixed">
     <parent link="base_footprint"/>
-    <child link="base_link" />
+    <child link="base_footprint" />
     <origin xyz="0 0.0 0.07" rpy="0 0 0.0"/>
   </joint> -->
-  <link name="base_link">
+  <link name="base_footprint">
     <visual>
       <origin xyz="0.097 0.276 0.19" rpy="3.14 0 -1.57"/>
@@ -31,5 +31,5 @@
   </link>
   <joint name="wheel_left_joint" type="continuous">
-    <parent link="base_link"/>
+    <parent link="base_footprint"/>
     <child link="wheel_left_link"/>
     <origin xyz="0.0 0.275 0.037" rpy="0.0 0.0 0"/>
@@ -59,5 +59,5 @@
   </link>
   <joint name="wheel_right_joint" type="continuous">
-    <parent link="base_link"/>
+    <parent link="base_footprint"/>
     <child link="wheel_right_link"/>
     <origin xyz="0.0 -0.275 0.037" rpy="0.0 0 0"/>
@@ -87,5 +87,5 @@
   </link>
   <joint name="caster_back_right_joint" type="fixed">
-    <parent link="base_link"/>
+    <parent link="base_footprint"/>
     <child link="caster_back_right_link"/>
     <origin xyz="-0.33 -0.148 0.06" rpy="0 0 0"/>
@@ -107,5 +107,5 @@
   </link>
   <joint name="caster_back_left_joint" type="fixed">
-    <parent link="base_link"/>
+    <parent link="base_footprint"/>
     <child link="caster_back_left_link"/>
     <origin xyz="-0.33 0.148 0.06" rpy="0 0 0"/>
@@ -127,5 +127,5 @@
   </link>
   <!-- <joint name="imu_joint" type="fixed">
-    <parent link="base_link"/>
+    <parent link="base_footprint"/>
     <child link="imu_link"/>
     <origin xyz="0.0 0 0.190" rpy="0 0 1.5758"/>
@@ -133,5 +133,5 @@
   <link name="imu_link"/> -->
   <joint name="scan_joint" type="fixed">
-    <parent link="base_link"/>
+    <parent link="base_footprint"/>
     <child link="base_scan"/>
     <origin xyz="0.06 0 0.230" rpy="0.0 0.0 0.0"/>
@@ -161,5 +161,5 @@
   <joint name="camera_joint" type="fixed">
     <origin xyz="0.07 0.0 0.63" rpy="0 0.7 0"/>
-    <parent link="base_link"/>
+    <parent link="base_footprint"/>
     <child link="camera_link"/>
   </joint>

Commit message: change urdf, ukf_template

File: Olaf_bot/Olaf_description/urdf/Olaf.urdf.g2.xacro (robot description, xacro)
@@ -2,5 +2,6 @@
 <robot name="Olaf" xmlns:xacro="http://ros.org/wiki/xacro">
   <xacro:include filename="$(find Olaf_description)/urdf/common_properties.xacro"/>
-  <!-- <link name="base_footprint"/>
+  <link name="base_footprint"/>
+<!--
   <joint name="base_joint" type="fixed">
     <parent link="base_footprint"/>
@@ -8,5 +9,5 @@
     <origin xyz="0 0.0 0.07" rpy="0 0 0.0"/>
   </joint> -->
-  <link name="base_footprint">
+  <!-- <link name="base_footprint">
     <visual>
       <origin xyz="0.097 0.276 0.19" rpy="3.14 0 -1.57"/>
@@ -29,12 +30,12 @@
                izz="2.0064271e-02" />
     </inertial>
-  </link>
-  <joint name="wheel_left_joint" type="continuous">
+  </link> -->
+  <!-- <joint name="wheel_left_joint" type="continuous">
     <parent link="base_footprint"/>
     <child link="wheel_left_link"/>
     <origin xyz="0.0 0.275 0.037" rpy="0.0 0.0 0"/>
     <axis xyz="0 1 0"/>
-  </joint>
-  <link name="wheel_left_link">
+  </joint> -->
+  <!-- <link name="wheel_left_link">
     <visual>
       <origin xyz="-0.1105 -0.06 0.1104" rpy="-1.57 0 0"/>
@@ -57,6 +58,6 @@
                izz="2.0712558e-03" />
       </inertial>
-  </link>
-  <joint name="wheel_right_joint" type="continuous">
+  </link> -->
+  <!-- <joint name="wheel_right_joint" type="continuous">
     <parent link="base_footprint"/>
     <child link="wheel_right_link"/>
@@ -85,6 +86,6 @@
                izz="2.0712558e-03" />
       </inertial>
-  </link>
-  <joint name="caster_back_right_joint" type="fixed">
+  </link> -->
+  <!-- <joint name="caster_back_right_joint" type="fixed">
     <parent link="base_footprint"/>
     <child link="caster_back_right_link"/>
@@ -125,5 +126,5 @@
                izz="0.000001" />
     </inertial>
-  </link>
+  </link> -->
   <!-- <joint name="imu_joint" type="fixed">
     <parent link="base_footprint"/>
@@ -135,5 +136,5 @@
     <parent link="base_footprint"/>
     <child link="base_scan"/>
-    <origin xyz="0.06 0 0.230" rpy="0.0 0.0 0.0"/>
+    <origin xyz="-0.07657 0 0.6439" rpy="0.0 0.0 0.0"/>
   </joint>
   <link name="base_scan">
@@ -159,5 +160,5 @@
     </inertial>
   </link>
-  <joint name="camera_joint" type="fixed">
+  <!-- <joint name="camera_joint" type="fixed">
     <origin xyz="0.07 0.0 0.63" rpy="0 0.7 0"/>
     <parent link="base_footprint"/>
@@ -190,4 +191,4 @@
     <child link="camera_rgb_optical_frame"/>
   </joint>
-  <link name="camera_rgb_optical_frame"/>
+  <link name="camera_rgb_optical_frame"/> -->
 </robot>

Commit message: only odom 11.28

File: Olaf_bot/Olaf_description/urdf/Olaf.urdf.g2.xacro (robot description, xacro)
@@ -3,6 +3,5 @@
   <xacro:include filename="$(find Olaf_description)/urdf/common_properties.xacro"/>
   <link name="base_footprint"/>
-<!--
-  <joint name="base_joint" type="fixed">
+  <!-- <joint name="base_joint" type="fixed">
     <parent link="base_footprint"/>
     <child link="base_footprint" />

Commit message: 12.7 change scan tf(temporary)

File: Olaf_bot/Olaf_description/urdf/Olaf.urdf.g2.xacro (robot description, xacro)
@@ -132,9 +132,10 @@
     <origin xyz="0.0 0 0.190" rpy="0 0 1.5758"/>
   </joint>
+  -0.07657 0.6439
   <link name="imu_link"/> -->
   <joint name="scan_joint" type="fixed">
     <parent link="base_footprint"/>
     <child link="base_scan"/>
-    <origin xyz="-0.07657 0 0.6439" rpy="0.0 0.0 0.0"/>
+    <origin xyz="0.09029 0 0.3235" rpy="0.0 0.0 0.0"/>
   </joint>
   <link name="base_scan">

Commit message: 12.09 Final

File: Olaf_bot/Olaf_description/urdf/Olaf.urdf.g2.xacro (robot description, xacro)
@@ -3,11 +3,10 @@
   <xacro:include filename="$(find Olaf_description)/urdf/common_properties.xacro"/>
   <link name="base_footprint"/>
-<!--
   <joint name="base_joint" type="fixed">
     <parent link="base_footprint"/>
-    <child link="base_footprint" />
+    <child link="base_link" />
     <origin xyz="0 0.0 0.07" rpy="0 0 0.0"/>
   </joint> -->
-  <!-- <link name="base_footprint">
+  <link name="base_link">
     <visual>
       <origin xyz="0.097 0.276 0.19" rpy="3.14 0 -1.57"/>
@@ -30,5 +29,5 @@
                izz="2.0064271e-02" />
     </inertial>
-  </link> -->
+  </link>
   <!-- <joint name="wheel_left_joint" type="continuous">
     <parent link="base_footprint"/>
@@ -127,14 +126,14 @@
     </inertial>
   </link> -->
-  <!-- <joint name="imu_joint" type="fixed">
-    <parent link="base_footprint"/>
+  <joint name="imu_joint" type="fixed">
+    <parent link="base_link"/>
     <child link="imu_link"/>
-    <origin xyz="0.0 0 0.190" rpy="0 0 1.5758"/>
+    <origin xyz="0.0 0 0.190" rpy="0 0 0"/>
   </joint>
   asfasdasdasfasdasa
   -0.07657 0.6439
-  <link name="imu_link"/> -->
+  <link name="imu_link"/>
   <joint name="scan_joint" type="fixed">
-    <parent link="base_footprint"/>
+    <parent link="base_link"/>
     <child link="base_scan"/>
     <origin xyz="0.09029 0 0.3235" rpy="0.0 0.0 0.0"/>

Commit message: 12.15 before topic

File: Olaf_bot/Olaf_description/urdf/Olaf.urdf.g2.xacro (robot description, xacro)
@@ -131,11 +131,9 @@
     <origin xyz="0.0 0 0.190" rpy="0 0 0"/>
   </joint>
-  asfasdasdasfasdasa
-  -0.07657 0.6439
   <link name="imu_link"/>
   <joint name="scan_joint" type="fixed">
     <parent link="base_link"/>
     <child link="base_scan"/>
-    <origin xyz="0.09029 0 0.3235" rpy="0.0 0.0 0.0"/>
+    <origin xyz="-0.07657 0 0.6439" rpy="0.0 0.0 0.0"/>
   </joint>
   <link name="base_scan">
